Commit message: adjust laser frame

File: magni_description/urdf/magni.urdf.xacro (robot description, xacro)
@@ -214,5 +214,5 @@
   <xacro:if value="${lidar_extrinsics_file != ''}">
     <xacro:property name="lidar_extrinsics" value="${load_yaml(lidar_extrinsics_file)}"/>
-    <xacro:ur50_lidar prefix="magni" name="laser" connected_to="base_link">
+    <xacro:ur50_lidar topic="scan" name="laser" connected_to="base_link">
       <!-- <origin xyz="${lidar_extrinsics['x']} ${lidar_extrinsics['y']} ${lidar_extrinsics['z']}"
         rpy="${lidar_extrinsics['roll']} ${lidar_extrinsics['pitch']} ${lidar_extrinsics['yaw']}"/> -->

File: magni_description/urdf/sensors/ur50_lidar.xacro (robot description, xacro)
@@ -1,5 +1,5 @@
 <?xml version="1.0" encoding="utf-8"?>
 <robot xmlns:xacro="http://wiki.ros.org/xacro">
-  <xacro:macro name="ur50_lidar" params="prefix:='' name:='' connected_to:=''  *origin">
+  <xacro:macro name="ur50_lidar" params="topic:='' name:='' connected_to:=''  *origin">
   <xacro:unless value="${connected_to == ''}">
     <joint name="${name}_joint" type="fixed">
@@ -55,5 +55,5 @@
       <!--<plugin name="gazebo_ros_head_hokuyo_controller" filename="libgazebo_ros_gpu_laser.so">-->
       <plugin name="gazebo_ros_head_hokuyo_controller" filename="libgazebo_ros_laser.so">
-        <topicName>${prefix}/scan</topicName>
+        <topicName>${topic}</topicName>
         <frameName>${name}</frameName>
       </plugin>

Commit message: first commit

File: magni_description/urdf/magni.urdf.xacro (robot description, xacro)
@@ -218,8 +218,9 @@
       <!-- <origin xyz="${lidar_extrinsics['x']} ${lidar_extrinsics['y']} ${lidar_extrinsics['z']}"
         rpy="${lidar_extrinsics['roll']} ${lidar_extrinsics['pitch']} ${lidar_extrinsics['yaw']}"/> -->
-<origin xyz="${lidar_extrinsics['x']+0.3} ${lidar_extrinsics['y']+0.05} ${lidar_extrinsics['z']}"
+<origin xyz="${lidar_extrinsics['x']} ${lidar_extrinsics['y']} ${lidar_extrinsics['z']}"
         rpy="${lidar_extrinsics['roll']} ${lidar_extrinsics['pitch']} ${lidar_extrinsics['yaw']}"/>
     </xacro:ur50_lidar>
   </xacro:if>
+<!--
    <joint name="added_joint" type="fixed">
       <origin xyz="-0.1 0 0.245" rpy="0 0 0" />
@@ -254,3 +255,4 @@
       </collision>
     </link>
+-->
 </robot>
